File: ASD2201.sch (EAGLE design)
At the start: 9 parts, among them J1 DF12-32-DP, J2 DF12-32-DS, J3 DM3D-SF, U1 XC6210B33, U2 TXB0104

Commit message: Update for Rev 2 Design
Parts:
- added R1, R2: 10.0K, tinycircuits:AS-ITM-00032
- added R3: 0.0, tinycircuits:AS-ITM-00076
- C2: PARTNUM AS-ITM-00049 -> (none)
- U1: value XC6210B33 -> XC6217A33; device tinycircuits:AS-ITM-00046 -> tinycircuits:AS-ITM-00249; PARTNO (none) -> AS-ITM-00249; VALUE (none) -> XC6217A33
Connections:
- new net N$1: J3.DAT2, R1.1
- new net N$2: J3.DAT1, R2.1
- new net N$9: R3.2, U1.NC/GO
- net GND: now also R3.1
- net VDD_SD: now also R1.2, R2.2
Other:
- note added: "2"
- note removed: "1"
- moved on the sheet: C3, C4
Changed lines of the file:
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@@
 <part name="U2" library="tinycircuits" deviceset="AS-ITM-00048" device="" value="TXB0104"/>
 <part name="J3" library="tinycircuits" deviceset="AS-ITM-00047" device="" value="DM3D-SF"/>
-<part name="U1" library="tinycircuits" deviceset="AS-ITM-00046" device="" value="XC6210B33"/>
+<part name="U1" library="tinycircuits" deviceset="AS-ITM-00249" device="" value="XC6217A33">
+<attribute name="PARTNO" value="AS-ITM-00249"/>
+<attribute name="VALUE" value="XC6217A33"/>
+</part>
 <part name="VCC3" library="tinycircuits" deviceset="VCC" device="" value="VCC"/>
 <part name="C3" library="tinycircuits" deviceset="AS-ITM-00008" device="" value="0.1uF">
@@
 <part name="GND6" library="tinycircuits" deviceset="GND" device=""/>
 <part name="C2" library="tinycircuits" deviceset="AS-ITM-00049" device="" value="47uF">
-<attribute name="PARTNUM" value="AS-ITM-00049"/>
 <attribute name="VALUE" value="47uF"/>
 </part>
 <part name="GND8" library="tinycircuits" deviceset="GND" device=""/>
 <part name="GND9" library="tinycircuits" deviceset="GND" device=""/>
+<part name="R1" library="tinycircuits" deviceset="AS-ITM-00032" device="" value="10.0K"/>
+<part name="R2" library="tinycircuits" deviceset="AS-ITM-00032" device="" value="10.0K"/>
+<part name="R3" library="tinycircuits" deviceset="AS-ITM-00076" device="" value="0.0"/>
+<part name="GND10" library="tinycircuits" deviceset="GND" device=""/>
 </parts>
 <sheets>
@@
 <text x="340.868" y="17.272" size="3.556" layer="94" font="vector">TinyShield - microSD Card</text>
 <text x="327.152" y="6.35" size="3.556" layer="94" font="vector">AS-SCH-ASD2201</text>
-<text x="416.56" y="6.858" size="3.556" layer="94" font="vector">1</text>
+<text x="416.56" y="6.858" size="3.556" layer="94" font="vector">2</text>
 <text x="299.72" y="142.24" size="3.81" layer="94" font="vector">TinyShield Expansion - Top</text>
 <text x="353.06" y="124.714" size="1.778" layer="91">IOREF</text>
@@
 <attribute name="VALUE" x="93.98" y="228.6" size="1.778" layer="96" rot="R180"/>
 </instance>
-<instance part="C3" gate="G$1" x="154.94" y="215.9" smashed="yes">
-<attribute name="NAME" x="158.242" y="215.519" size="1.778" layer="95"/>
-<attribute name="VALUE" x="158.242" y="213.233" size="1.778" layer="96"/>
+<instance part="C3" gate="G$1" x="167.64" y="215.9" smashed="yes">
+<attribute name="NAME" x="170.942" y="215.519" size="1.778" layer="95"/>
+<attribute name="VALUE" x="170.942" y="213.233" size="1.778" layer="96"/>
 </instance>
 <instance part="GND2" gate="1" x="116.84" y="208.28"/>
-<instance part="C4" gate="G$1" x="170.18" y="215.9" smashed="yes">
-<attribute name="NAME" x="173.228" y="215.519" size="1.778" layer="95"/>
-<attribute name="VALUE" x="173.228" y="213.233" size="1.778" layer="96"/>
+<instance part="C4" gate="G$1" x="182.88" y="215.9" smashed="yes">
+<attribute name="NAME" x="185.928" y="215.519" size="1.778" layer="95"/>
+<attribute name="VALUE" x="185.928" y="213.233" size="1.778" layer="96"/>
 </instance>
 <instance part="VCC4" gate="VCC" x="195.58" y="134.62" smashed="yes">
@@
 <instance part="GND3" gate="1" x="93.98" y="104.14"/>
 <instance part="GND4" gate="1" x="193.04" y="106.68"/>
-<instance part="GND5" gate="1" x="154.94" y="205.74"/>
-<instance part="GND6" gate="1" x="170.18" y="205.74"/>
+<instance part="GND5" gate="1" x="167.64" y="205.74"/>
+<instance part="GND6" gate="1" x="182.88" y="205.74"/>
 <instance part="C2" gate="G$1" x="91.44" y="215.9" smashed="yes">
 <attribute name="NAME" x="94.742" y="215.519" size="1.778" layer="95"/>
@@
 <instance part="GND8" gate="1" x="104.14" y="205.74"/>
 <instance part="GND9" gate="1" x="91.44" y="205.74"/>
+<instance part="R1" gate="G$1" x="106.68" y="132.08"/>
+<instance part="R2" gate="G$1" x="106.68" y="106.68"/>
+<instance part="R3" gate="G$1" x="154.94" y="208.28" rot="R90"/>
+<instance part="GND10" gate="1" x="154.94" y="198.12"/>
 </instances>
 <busses>
@@
 <pinref part="GND5" gate="1" pin="GND"/>
 <pinref part="C3" gate="G$1" pin="2"/>
-<wire x1="154.94" y1="208.28" x2="154.94" y2="210.82" width="0.1524" layer="91"/>
+<wire x1="167.64" y1="208.28" x2="167.64" y2="210.82" width="0.1524" layer="91"/>
 </segment>
 <segment>
 <pinref part="C4" gate="G$1" pin="2"/>
 <pinref part="GND6" gate="1" pin="GND"/>
-<wire x1="170.18" y1="210.82" x2="170.18" y2="208.28" width="0.1524" layer="91"/>
+<wire x1="182.88" y1="210.82" x2="182.88" y2="208.28" width="0.1524" layer="91"/>
 </segment>
 <segment>
@@
 <pinref part="C1" gate="G$1" pin="2"/>
 <wire x1="104.14" y1="208.28" x2="104.14" y2="210.82" width="0.1524" layer="91"/>
+</segment>
+<segment>
+<pinref part="R3" gate="G$1" pin="1"/>
+<wire x1="154.94" y1="203.2" x2="154.94" y2="200.66" width="0.1524" layer="91"/>
+<pinref part="GND10" gate="1" pin="GND"/>
 </segment>
 </net>
@@
 <junction x="160.02" y="127"/>
 <label x="137.16" y="127.508" size="1.778" layer="95"/>
+<pinref part="R1" gate="G$1" pin="2"/>
+<wire x1="111.76" y1="132.08" x2="114.3" y2="132.08" width="0.1524" layer="91"/>
+<wire x1="114.3" y1="132.08" x2="114.3" y2="127" width="0.1524" layer="91"/>
+<junction x="114.3" y="127"/>
+<pinref part="R2" gate="G$1" pin="2"/>
+<wire x1="111.76" y1="106.68" x2="160.02" y2="106.68" width="0.1524" layer="91"/>
+<wire x1="160.02" y1="106.68" x2="160.02" y2="111.76" width="0.1524" layer="91"/>
+<junction x="160.02" y="111.76"/>
 </segment>
 <segment>
 <pinref part="U1" gate="G$1" pin="VOUT"/>
 <pinref part="C4" gate="G$1" pin="1"/>
-<wire x1="170.18" y1="218.44" x2="170.18" y2="220.98" width="0.1524" layer="91"/>
-<wire x1="170.18" y1="220.98" x2="154.94" y2="220.98" width="0.1524" layer="91"/>
+<wire x1="182.88" y1="218.44" x2="182.88" y2="220.98" width="0.1524" layer="91"/>
+<wire x1="182.88" y1="220.98" x2="167.64" y2="220.98" width="0.1524" layer="91"/>
 <pinref part="C3" gate="G$1" pin="1"/>
-<wire x1="154.94" y1="220.98" x2="147.32" y2="220.98" width="0.1524" layer="91"/>
-<wire x1="154.94" y1="218.44" x2="154.94" y2="220.98" width="0.1524" layer="91"/>
-<label x="160.02" y="221.488" size="1.778" layer="95"/>
-<junction x="154.94" y="220.98"/>
+<wire x1="167.64" y1="220.98" x2="147.32" y2="220.98" width="0.1524" layer="91"/>
+<wire x1="167.64" y1="218.44" x2="167.64" y2="220.98" width="0.1524" layer="91"/>
+<label x="172.72" y="221.488" size="1.778" layer="95"/>
+<junction x="167.64" y="220.98"/>
 </segment>
 </net>
@@
 </segment>
 </net>
+<net name="N$1" class="0">
+<segment>
+<pinref part="J3" gate="G$1" pin="DAT2"/>
+<wire x1="91.44" y1="127" x2="96.52" y2="127" width="0.1524" layer="91"/>
+<wire x1="96.52" y1="127" x2="96.52" y2="132.08" width="0.1524" layer="91"/>
+<pinref part="R1" gate="G$1" pin="1"/>
+<wire x1="96.52" y1="132.08" x2="101.6" y2="132.08" width="0.1524" layer="91"/>
+</segment>
+</net>
+<net name="N$2" class="0">
+<segment>
+<pinref part="J3" gate="G$1" pin="DAT1"/>
+<wire x1="91.44" y1="109.22" x2="99.06" y2="109.22" width="0.1524" layer="91"/>
+<wire x1="99.06" y1="109.22" x2="99.06" y2="106.68" width="0.1524" layer="91"/>
+<pinref part="R2" gate="G$1" pin="1"/>
+<wire x1="99.06" y1="106.68" x2="101.6" y2="106.68" width="0.1524" layer="91"/>
+</segment>
+</net>
+<net name="N$9" class="0">
+<segment>
+<pinref part="R3" gate="G$1" pin="2"/>
+<pinref part="U1" gate="G$1" pin="NC/GO"/>
+<wire x1="154.94" y1="213.36" x2="154.94" y2="215.9" width="0.1524" layer="91"/>
+<wire x1="154.94" y1="215.9" x2="147.32" y2="215.9" width="0.1524" layer="91"/>
+</segment>
+</net>
