File: design_files/ASD2201.sch (EAGLE design)
At the start: 12 parts, among them J1 DF12-32-DP, J2 DF12-32-DS, J3 DM3D-SF, U1 XC6217A33, U2 TXB0104

Commit message: update format
Other:
- note added: "Hand Populated: -"
- note added: "Hand Soldered: -"
- note added: "Non Populated: -"
- note added: "Variant: Standard - R"
Changed lines of the file:
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@@
 <layer number="46" name="Milling" color="3" fill="1" visible="no" active="no"/>
 <layer number="47" name="Measures" color="7" fill="1" visible="no" active="no"/>
-<layer number="48" name="Document" color="7" fill="1" visible="no" active="no"/>
+<layer number="48" name="Document" color="10" fill="1" visible="no" active="no"/>
 <layer number="49" name="Reference" color="7" fill="1" visible="no" active="no"/>
 <layer number="50" name="ReferenceLS" color="7" fill="1" visible="no" active="no"/>
@@
 <text x="157.48" y="144.78" size="3.81" layer="94" font="vector">Level Shifter</text>
 <text x="45.72" y="147.32" size="3.81" layer="94" font="vector">microSD Card Connector</text>
+<text x="60.96" y="68.58" size="1.778" layer="96">Non Populated: -</text>
+<text x="60.96" y="66.04" size="1.778" layer="96">Hand Populated: -</text>
+<text x="60.96" y="63.5" size="1.778" layer="96">Hand Soldered: -</text>
+<text x="60.96" y="71.12" size="1.778" layer="96">Variant: Standard - R</text>
 </plain>
 <instances>
